Commit message: Update SO101 gripper mass properties
Update inertial properties for SO101 follower arm gripper parts based on
updated CAD models:

- Moving Jaw Follower SO101:
  - Mass: 0.012 kg → 0.09 kg
  - Updated center of mass and moment of inertia tensor

- Wrist Roll Follower SO101:
  - Mass: 0.087 kg → 0.044 kg
  - Updated center of mass and moment of inertia tensor

Changes applied to both MuJoCo XML and URDF simulation files for new and
old calibration variants.

File: Simulation/SO101/so101_new_calib.urdf (robot description, URDF)
Before this commit: robot so101_new_calib, 8 links, 7 joints
Links:
- link gripper_link: mass 0.087 -> 0.044
- link moving_jaw_so101_v1_link: mass 0.012 -> 0.09

File: Simulation/SO101/so101_old_calib.urdf (robot description, URDF)
Before this commit: robot so101_old_calib, 7 links, 6 joints
Links:
- link gripper: mass 0.087 -> 0.044
- link jaw: mass 0.012 -> 0.09
